File: MainPCB/MainPCB.kicad_sch (KiCad schematic)
At the start: 0 parts

Commit message: Schaltplan erstellt
Parts:
- added C1, C2, C5, C6: 4u7, Capacitor_SMD:C_0805_2012Metric, symbol Device:C
- added C3, C4: 100n, Capacitor_SMD:C_0603_1608Metric, symbol Device:C
- added IC1: AP7361EA-33E-13, symbol SamacSys_Parts:AP7361EA-33E-13
- added J1: 1757242, SamacSys_Parts:1757242, symbol SamacSys_Parts:1757242
- added J2: 1757255, SamacSys_Parts:1757255, symbol SamacSys_Parts:1757255
- added J3: Conn_01x10, symbol Connector_Generic:Conn_01x11
- added J4, J5, J6, J7, J8: 2466267-1, SamacSys_Parts:24662671, symbol SamacSys_Parts:2466267-1
- added R1, R2: 150, Resistor_SMD:R_0603_1608Metric, symbol Device:R
- added R3: tbd, symbol Device:R
- added U2: LM78M05_TO220, Package_TO_SOT_THT:TO-220-3_Vertical, symbol Regulator_Linear:LM78M05_TO220
Connections:
- new net: J1.2, J6.1, J7.1, R3.1
- new net +12V: C2.1, J3.2 (Pin_2), J7.2, J7.3, J7.4, J7.5, R3.2, U2.1 (VI)
- new net +3.3V: C5.1, IC1.3 (OUT), J3.3 (Pin_3)
- new net +5V: C1.1, C6.1, IC1.1 (IN), U2.3 (VO)
- new net 0V: J2.1, J3.11 (Pin_11)
- new net 400V: J2.3, J3.1 (Pin_1)
- new net GND: C1.2, C2.2, C3.2, C4.2, C5.2, C6.2, IC1.2 (GND_1), IC1.4 (GND_2), J1.1, J3.4 (Pin_4), J4.2, J4.3, J4.4, J4.5, J5.2, J5.3, J5.4, J5.5, J6.2, J6.3, J6.4, J6.5, J8.2, J8.3, J8.4, J8.5, U2.2 (GND)
- new net I_VOUT: J3.9 (Pin_9), R1.2
- new net I_VREF: J3.10 (Pin_10), R2.2
- new net Mikrocontroller/ADCINA2: C3.1, R1.1
- new net Mikrocontroller/ADCINA3: C4.1, R2.1
- new net PWM_CLAMPING_1: J4.1
- new net PWM_CLAMPING_2: J5.1
- new net PWM_S11: J3.5 (Pin_5), J8.1
- new net PWM_S12: J3.6 (Pin_6)
- new net PWM_S21: J3.7 (Pin_7)
- new net PWM_S22: J3.8 (Pin_8)
- no-connect marks 0 -> 1
Other:
- added sheet Mikrocontroller (Mikrocontroller.kicad_sch)
- note added: "12V Eingang mit BNC-Stecker zum Messen"
- note added: "400V Eingang"
- note added: "FOOTPRINT FEHLT"
- note added: "Lötverbindungen zur Transistorplatine"
- note added: "Mikrocontroller"
- note added: "PWM BNC Steckverbindung"
- note added: "Spannungsversorgung für Mikrocontroller"
- company: (none) -> TU Berlin - Fachgebiet Leistungselektronik
- title: (none) -> Hauptplatine
